File: hardware/carrier/intercom-carrier.kicad_pcb (KiCad board)
At the start: 2 copper layers, 0 parts

Commit message: hardware: carrier PCB layout (rev A) for the ESP32-P4-ETH
Two 1x20 sockets for the P4's Pico-style header, four button/LED channels
along the bottom edge, GND pours on both layers, four M3 holes.
DRC: 0 errors, 0 unconnected. Gerbers, PDFs and BOM in carrier/export/.
README and notes now describe the board actually used (P4-ETH, no WiFi).

Co-Authored-By: Claude Opus 5.5 <noreply@anthropic.com>
Parts:
- added C1: 100nF, Capacitor_THT:C_Disc_D3.0mm_W1.6mm_P2.50mm, F.Cu at (142.8, 131.2)
- added C2: 100nF, Capacitor_THT:C_Disc_D3.0mm_W1.6mm_P2.50mm, F.Cu at (187.2, 131.2)
- added C3: 100nF, Capacitor_THT:C_Disc_D3.0mm_W1.6mm_P2.50mm, F.Cu at (165.0, 131.2)
- added C4: 100nF, Capacitor_THT:C_Disc_D3.0mm_W1.6mm_P2.50mm, F.Cu at (120.6, 131.2)
- added C5: 10uF, Capacitor_THT:CP_Radial_D5.0mm_P2.00mm, F.Cu at (142.1, 144.5)
- added H1: MountingHole_3.2mm_M3, MountingHole:MountingHole_3.2mm_M3, F.Cu at (103.0, 103.5)
- added H2: MountingHole_3.2mm_M3, MountingHole:MountingHole_3.2mm_M3, F.Cu at (187.2, 121.0)
- added H3: MountingHole_3.2mm_M3, MountingHole:MountingHole_3.2mm_M3, F.Cu at (121.8, 144.3)
- added H4: MountingHole_3.2mm_M3, MountingHole:MountingHole_3.2mm_M3, F.Cu at (166.2, 144.3)
- added J1: P4 pins 1-20, Connector_PinSocket_2.54mm:PinSocket_1x20_P2.54mm_Vertical, F.Cu at (179.3, 103.6)
- added J2: Button 1 (JST-XH), Connector_JST:JST_XH_B4B-XH-A_1x04_P2.50mm_Vertical, F.Cu at (129.2, 144.0)
- added J3: Button 2 (JST-XH), Connector_JST:JST_XH_B4B-XH-A_1x04_P2.50mm_Vertical, F.Cu at (173.6, 144.0)
- added J4: Button 3 (JST-XH), Connector_JST:JST_XH_B4B-XH-A_1x04_P2.50mm_Vertical, F.Cu at (151.4, 144.0)
- added J5: Button 4 (JST-XH), Connector_JST:JST_XH_B4B-XH-A_1x04_P2.50mm_Vertical, F.Cu at (107.0, 144.0)
- added J6: Spare GPIO2/3, Connector_PinHeader_2.54mm:PinHeader_1x04_P2.54mm_Vertical, F.Cu at (187.8, 106.5)
- added J7: P4 pins 21-40, Connector_PinSocket_2.54mm:PinSocket_1x20_P2.54mm_Vertical, F.Cu at (131.1, 121.4)
- added Q1: BC547, Package_TO_SOT_THT:TO-92_Inline, F.Cu at (131.1, 135.5)
- added Q2: BC547, Package_TO_SOT_THT:TO-92_Inline, F.Cu at (175.4, 135.5)
- added Q3: BC547, Package_TO_SOT_THT:TO-92_Inline, F.Cu at (153.2, 135.5)
- added Q4: BC547, Package_TO_SOT_THT:TO-92_Inline, F.Cu at (108.8, 135.5)
- added R1: 1k, Resistor_THT:R_Axial_DIN0207_L6.3mm_D2.5mm_P7.62mm_Horizontal, F.Cu at (142.8, 127.5)
- added R10: 10k, Resistor_THT:R_Axial_DIN0207_L6.3mm_D2.5mm_P7.62mm_Horizontal, F.Cu at (176.7, 131.0)
- added R11: 10k, Resistor_THT:R_Axial_DIN0207_L6.3mm_D2.5mm_P7.62mm_Horizontal, F.Cu at (154.5, 131.0)
- added R12: 10k, Resistor_THT:R_Axial_DIN0207_L6.3mm_D2.5mm_P7.62mm_Horizontal, F.Cu at (110.1, 131.0)
- added R13: 0R, Resistor_THT:R_Axial_DIN0207_L6.3mm_D2.5mm_P7.62mm_Horizontal, F.Cu at (124.1, 139.3)
- added R14: 0R, Resistor_THT:R_Axial_DIN0207_L6.3mm_D2.5mm_P7.62mm_Horizontal, F.Cu at (168.5, 139.3)
- added R15: 0R, Resistor_THT:R_Axial_DIN0207_L6.3mm_D2.5mm_P7.62mm_Horizontal, F.Cu at (146.3, 139.3)
- added R16: 0R, Resistor_THT:R_Axial_DIN0207_L6.3mm_D2.5mm_P7.62mm_Horizontal, F.Cu at (101.9, 139.3)
- added R2: 1k, Resistor_THT:R_Axial_DIN0207_L6.3mm_D2.5mm_P7.62mm_Horizontal, F.Cu at (187.2, 127.5)
- added R3: 1k, Resistor_THT:R_Axial_DIN0207_L6.3mm_D2.5mm_P7.62mm_Horizontal, F.Cu at (165.0, 127.5)
- added R4: 1k, Resistor_THT:R_Axial_DIN0207_L6.3mm_D2.5mm_P7.62mm_Horizontal, F.Cu at (120.6, 127.5)
- added R5: 1k, Resistor_THT:R_Axial_DIN0207_L6.3mm_D2.5mm_P7.62mm_Horizontal, F.Cu at (124.7, 127.5)
- added R6: 1k, Resistor_THT:R_Axial_DIN0207_L6.3mm_D2.5mm_P7.62mm_Horizontal, F.Cu at (169.1, 127.5)
- added R7: 1k, Resistor_THT:R_Axial_DIN0207_L6.3mm_D2.5mm_P7.62mm_Horizontal, F.Cu at (146.9, 127.5)
- added R8: 1k, Resistor_THT:R_Axial_DIN0207_L6.3mm_D2.5mm_P7.62mm_Horizontal, F.Cu at (102.5, 127.5)
- added R9: 10k, Resistor_THT:R_Axial_DIN0207_L6.3mm_D2.5mm_P7.62mm_Horizontal, F.Cu at (132.3, 131.0)
Routing:
- net +5V: track 0.00 -> 115.4 mm
- net /LED4_GPIO5: track 0.00 -> 75.3 mm
- net /SPARE_GPIO2: track 0.00 -> 52.3 mm
- net /SPARE_GPIO3: track 0.00 -> 50.7 mm
- net /BTN4_GPIO23: track 0.00 -> 45.7 mm
- net /LED2_GPIO33: track 0.00 -> 36.4 mm, vias 0 -> 1
- net /BTN2_GPIO20: track 0.00 -> 30.4 mm
- net /LED3_GPIO4: track 0.00 -> 27.6 mm
- net /BTN1_GPIO22: track 0.00 -> 26.0 mm
- net /LED1_GPIO32: track 0.00 -> 25.2 mm
- net /BTN1_SW: track 0.00 -> 16.9 mm
- net /BTN4_SW: track 0.00 -> 16.9 mm
- net /BTN3_SW: track 0.00 -> 16.9 mm
- net /BTN2_SW: track 0.00 -> 16.9 mm
- net /LED1_COL: track 0.00 -> 10.8 mm
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- added copper zone on B.Cu, net GND
- added copper zone on F.Cu, net GND
Other:
- board outline added: 90 x 48 mm
- board text added: "BTN1"
- board text added: "BTN2"
- board text added: "BTN3"
- board text added: "BTN4"
- board text added: "ESP32-P4-ETH: RJ45 this end"
- board text added: "GPIO2 GPIO3 GND GND"
- board text added: "USB-C this end"
- board text added: "intercom carrier rev A — JST: 1 +5V, 2 LED-, 3 SW, 4 GND"

Commit message: carrier: number buttons 1-4 left to right; PTT moves to GPIO23
The channels were placed in the order their GPIOs leave the header (clean,
crossing-free routing) but kept the old numbers, so the silkscreen read
BTN4 BTN1 BTN3 BTN2. Renumbered the nets and parts instead of the copper:
buttons 1-4 are GPIO23/22/21/20, LED rings GPIO5/32/4/33. PTT (button 1)
is now GPIO23 in lanicom-p4.yaml. DRC 0 errors, 0 unconnected.

Co-Authored-By: Claude Opus 5.5 <noreply@anthropic.com>
Claude-Session: https://claude.ai/code/session_01CWRFtk6j7DsJxLJbKSRr78
Parts:
- J2: renamed from J5; value Button 4 (JST-XH) -> Button 1 (JST-XH)
- J3: renamed from J2; value Button 1 (JST-XH) -> Button 2 (JST-XH)
- J5: renamed from J3; value Button 2 (JST-XH) -> Button 4 (JST-XH)
- renumbered C4 to C1, C1 to C2, C2 to C4, Q4 to Q1, Q1 to Q2, Q2 to Q4, R4 to R1, R9 to R10, R10 to R12, R16 to R13, R13 to R14, R14 to R16, R1 to R2, R2 to R4, R8 to R5, R5 to R6, R6 to R8, R12 to R9
Connections:
- net /BTN1_GPIO22 renamed /BTN2_GPIO22
- net /BTN2_GPIO20 renamed /BTN4_GPIO20
- net /BTN4_GPIO23 renamed /BTN1_GPIO23
- net /LED1_GPIO32 renamed /LED2_GPIO32
- net /LED2_GPIO33 renamed /LED4_GPIO33
- net /LED4_GPIO5 renamed /LED1_GPIO5
- J2 pad 2: /LED4_K -> /LED1_K
- J2 pad 3: /BTN4_SW -> /BTN1_SW
- J3 pad 2: /LED1_K -> /LED2_K
- J3 pad 3: /BTN1_SW -> /BTN2_SW
- J5 pad 2: /LED2_K -> /LED4_K
- J5 pad 3: /BTN2_SW -> /BTN4_SW
- Q1 pad 1: /LED4_COL -> /LED1_COL
- Q2 pad 1: /LED1_COL -> /LED2_COL
- Q4 pad 1: /LED2_COL -> /LED4_COL
- R1 pad 2: /BTN4_SW -> /BTN1_SW
- R13 pad 1: /LED4_COL -> /LED1_COL
- R13 pad 2: /LED4_K -> /LED1_K
- R14 pad 1: /LED1_COL -> /LED2_COL
- R14 pad 2: /LED1_K -> /LED2_K
- R16 pad 1: /LED2_COL -> /LED4_COL
- R16 pad 2: /LED2_K -> /LED4_K
- R2 pad 2: /BTN1_SW -> /BTN2_SW
- R4 pad 2: /BTN2_SW -> /BTN4_SW

Commit message: carrier: J6 silkscreen, one label per pin in the right order
The old rotated label read GND at pin 1; pin 1 is GPIO2.

Co-Authored-By: Claude Opus 5.5 <noreply@anthropic.com>
Claude-Session: https://claude.ai/code/session_01CWRFtk6j7DsJxLJbKSRr78
Other:
- board text added: "GND"
- board text added: "GPIO2"
- board text added: "GPIO3"
- board text removed: "GPIO2 GPIO3 GND GND"
