File: hardware/carrier/intercom-carrier.kicad_sch (KiCad schematic)
At the start: 31 parts, among them J1 Host P6 (2x20 socket), J2 Button 1 (JST-XH), J3 Button 2 (JST-XH), J4 Button 3 (JST-XH), J5 Button 4 (JST-XH), J6 Spare GPIO2/3, Q1 BC547, Q2 BC547, Q3 BC547, Q4 BC547

Commit message: hardware: carrier PCB layout (rev A) for the ESP32-P4-ETH
Two 1x20 sockets for the P4's Pico-style header, four button/LED channels
along the bottom edge, GND pours on both layers, four M3 holes.
DRC: 0 errors, 0 unconnected. Gerbers, PDFs and BOM in carrier/export/.
README and notes now describe the board actually used (P4-ETH, no WiFi).

Co-Authored-By: Claude Opus 5.5 <noreply@anthropic.com>
Parts:
- removed J1: Host P6 (2x20 socket), Connector_PinSocket_2.54mm:PinSocket_2x20_P2.54mm_Vertical, symbol Connector_Generic:Conn_02x20_Odd_Even
- added J1: P4 pins 1-20, Connector_PinSocket_2.54mm:PinSocket_1x20_P2.54mm_Vertical, symbol Connector_Generic:Conn_01x20
- added J7: P4 pins 21-40, Connector_PinSocket_2.54mm:PinSocket_1x20_P2.54mm_Vertical, symbol Connector_Generic:Conn_01x20
Connections:
- net +5V: now also J7.19 (Pin_19)
- net BTN1_GPIO22: now also J7.12 (Pin_12)
- net BTN2_GPIO20: now also J7.15 (Pin_15)
- net BTN3_GPIO21: now also J7.14 (Pin_14)
- net BTN4_GPIO23: now also J7.11 (Pin_11)
- net GND: now also J1.13 (Pin_13), J1.18 (Pin_18), J1.3 (Pin_3), J1.8 (Pin_8), J7.13 (Pin_13), J7.18 (Pin_18), J7.3 (Pin_3), J7.8 (Pin_8)
- net LED1_GPIO32: now also J7.6 (Pin_6)
- net LED2_GPIO33: now also J7.5 (Pin_5)
- net LED3_GPIO4: now also J1.12 (Pin_12)
- net LED4_GPIO5: now also J1.11 (Pin_11)
- net SPARE_GPIO2: now also J1.15 (Pin_15)
- net SPARE_GPIO3: now also J1.14 (Pin_14)
- no-connect marks 20 -> 21
Other:
- note added: "Base board for the Waveshare ESP32-P4-ETH / -POE-ETH: the module plugs in from above (header P1, Pico layout, rows 17.78 mm apart). J1 = P4 pins 1-20, J7 = P4 pins 21-40. +5V = VSYS (P4 pin 39). The PoE module sits on top of the P4. All parts through-hole. ESPHome: buttons GPIO22/20/21/23 INPUT_PULLUP, inverted (pressed = low); LEDs GPIO32/33/4/5 via LEDC (PWM). Button connectors (JST-XH): 1 = LE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"
- note removed: "Intercom carrier, rev A, 2026-10-06 (Intercom boerderij) Plugs onto header P6 of the Waveshare ESP32-P4-WIFI6-POE-ETH. All parts through-hole. ESPHome: buttons GPIO22/20/21/23 INPUT_PULLUP, inverted (pressed = low). LEDs GPIO32/33/4/5 via LEDC (PWM), active high. Button connectors (JST-XH): 1 = LED+ (+5V), 2 = LED-, 3 = switch, 4 = GND. R13-R16: fit 0R, or a resistor once the ring current at 5 V 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"
- title: (none) -> Intercom carrier

Commit message: carrier: number buttons 1-4 left to right; PTT moves to GPIO23
The channels were placed in the order their GPIOs leave the header (clean,
crossing-free routing) but kept the old numbers, so the silkscreen read
BTN4 BTN1 BTN3 BTN2. Renumbered the nets and parts instead of the copper:
buttons 1-4 are GPIO23/22/21/20, LED rings GPIO5/32/4/33. PTT (button 1)
is now GPIO23 in lanicom-p4.yaml. DRC 0 errors, 0 unconnected.

Co-Authored-By: Claude Opus 5.5 <noreply@anthropic.com>
Claude-Session: https://claude.ai/code/session_01CWRFtk6j7DsJxLJbKSRr78
Parts:
- J2: renamed from J5; value Button 4 (JST-XH) -> Button 1 (JST-XH)
- J3: renamed from J2; value Button 1 (JST-XH) -> Button 2 (JST-XH)
- J5: renamed from J3; value Button 2 (JST-XH) -> Button 4 (JST-XH)
- renumbered C4 to C1, C1 to C2, C2 to C4, Q4 to Q1, Q1 to Q2, Q2 to Q4, R4 to R1, R9 to R10, R10 to R12, R16 to R13, R13 to R14, R14 to R16, R1 to R2, R2 to R4, R8 to R5, R5 to R6, R6 to R8, R12 to R9
Connections:
- net BTN1_SW: now also J2.3 (Pin_3), R1.2; no longer J3.3 (Pin_3), R2.2
- net BTN2_SW: now also J3.3 (Pin_3), R2.2; no longer J5.3 (Pin_3), R4.2
- net BTN4_SW: now also J5.3 (Pin_3), R4.2; no longer J2.3 (Pin_3), R1.2
- net LED1_COL: now also Q1.1 (C), R13.1; no longer Q2.1 (C), R14.1
- net LED1_K: now also J2.2 (Pin_2), R13.2; no longer J3.2 (Pin_2), R14.2
- net LED2_COL: now also Q2.1 (C), R14.1; no longer Q4.1 (C), R16.1
- net LED2_K: now also J3.2 (Pin_2), R14.2; no longer J5.2 (Pin_2), R16.2
- net LED4_COL: now also Q4.1 (C), R16.1; no longer Q1.1 (C), R13.1
- net LED4_K: now also J5.2 (Pin_2), R16.2; no longer J2.2 (Pin_2), R13.2
- net BTN1_GPIO22 renamed BTN2_GPIO22
- net BTN2_GPIO20 renamed BTN4_GPIO20
- net BTN4_GPIO23 renamed BTN1_GPIO23
- net LED1_GPIO32 renamed LED2_GPIO32
- net LED2_GPIO33 renamed LED4_GPIO33
- net LED4_GPIO5 renamed LED1_GPIO5

Commit message: carrier rev B: off switch connector J8 on 3V3_EN
J8 (JST-XH 2-pin, 1 = 3V3_EN / P4 pin 37, 2 = GND) with C6 100 nF across it,
in the bottom-right corner next to the button JSTs. J5 moved 1.1 mm left to
make room; its tracks are re-routed. 3V3_EN runs on B.Cu from J7.17.
Mounting holes and J6 are unchanged, so the enclosure is too.
ERC clean, DRC 0 errors / 0 unconnected. carrier/export/ is still rev A.

Co-Authored-By: Claude Opus 5.5 <noreply@anthropic.com>
Parts:
- added C6: 100nF, Capacitor_THT:C_Disc_D3.0mm_W1.6mm_P2.50mm, symbol Device:C
- added J8: Off switch (JST-XH), Connector_JST:JST_XH_B2B-XH-A_1x02_P2.50mm_Vertical, symbol Connector_Generic:Conn_01x02
Connections:
- net GND: now also C6.2, J8.2 (Pin_2)
- net 3V3_EN: now reaches J7.17 (Pin_17)
- net 3V3_EN: now also C6.1, J8.1 (Pin_1)
- no-connect marks 21 -> 20
